Commit message: Unspringed springs, symmetrised brain, and automatic blockage generation

File: src/pipebot_description/urdf/sprintbot.urdf (robot description, URDF)
Before this commit: robot sprintbot_basic_collisions, 6 links, 5 joints
Joints:
- joint back_spring: limit lower=-0.01 upper=0.02 effort=0 velocity=0 -> (none); origin xyz=-0.12 0 -0.1 rpy=0 0 0 -> xyz=-0.12 0 -0.08 rpy=0 0 0; type prismatic -> fixed
- joint front_spring: limit lower=-0.01 upper=0.02 effort=0 velocity=0 -> (none); origin xyz=0.12 0 -0.1 rpy=0 0 0 -> xyz=0.12 0 -0.08 rpy=0 0 0; type prismatic -> fixed
